Commit message: feat(sim): RobotBuilder, ball-script UI, and URDF wiring
- Add RobotBuilder with competition mount presets
- Wire URDF meshes into the viewer (control still uses competition Arm)
- Update competition_arm.urdf link lengths to match the short arm
- Add / improve on-screen panel controls for ball scripts
- Improve viewer overlays and camera helpers for swing debugging
- Small telemetry and session wiring updates for the new builder path

File: assets/robots/competition_arm.urdf (robot description, URDF)
Before this commit: robot pingpong_competition_arm, 4 links, 3 joints
Links:
- link base_link: geometry visual cylinder length=0.05 radius=0.06
- link link1: geometry visual cylinder length=0.16 radius=0.025
- link link2: geometry visual cylinder length=0.14 radius=0.022
- link racket_link: geometry visual box size=0.12 0.14 0.010
Joints:
- joint joint_elbow: origin xyz=0 0.30 0 rpy=0 0 0 -> xyz=0 0.14 0 rpy=0 0 0
- joint joint_shoulder: origin xyz=0 0.35 0 rpy=0 0 0 -> xyz=0 0.16 0 rpy=0 0 0
- joint joint_yaw: origin xyz=-1.35 0.76 -1.1 rpy=0 0 0 -> xyz=0 0 0 rpy=0 0 0
