Commit message: fix(robots): correct 4-dof link masses to measured/spec values
CAD-exported masses were unreliable (e.g. paddle at 2.4kg, MX-64R at
568g). Replace mass with real measurements/datasheet values for
arm_v9_1, arm2_v2_1, pingpong_paddle_v5_1, racket_joint_v8_1, and the
MX-28T/MX-64R servos, scaling each link's inertia tensor by the same
mass ratio since geometry is unchanged. Applied identically to both
all-4-export.urdf (runtime) and all-4-export.xacro (CAD source) to
keep them in sync. Aluminum brackets left untouched pending CAD
density confirmation; racket_joint_v8_1 flagged with a TODO since the
measured mass is from a v9 part not yet reflected in this mesh.

Co-Authored-By: Claude Sonnet 5 <noreply@anthropic.com>

File: assets/robots/4-dof/urdf/all-4-export.urdf (robot description, URDF)
Before this commit: robot all-4-export, 17 links, 16 joints
Links:
- link MX-28T_R_v1_1: mass 0.3395854409997755 -> 0.072
- link MX-28T_R_v1__1__1: mass 0.3395854409997755 -> 0.072
- link MX-64R_v1_1: mass 0.5685307980275295 -> 0.126
- link MX-64R_v1__1__1: mass 0.5685307980275295 -> 0.126
- link MX-64R_v1__2__1: mass 0.5685307980275295 -> 0.126
- link arm2_v2_1: mass 0.1756574712319971 -> 0.0217
- link arm_v9_1: mass 0.24310181617070015 -> 0.027
- link pingpong_paddle_v5_1: mass 2.4030890000623666 -> 0.1729
- link racket_joint_v8_1: mass 0.3222277062125533 -> 0.0265

File: assets/robots/4-dof/urdf/all-4-export.xacro (robot description, xacro)
@@ -27,6 +27,7 @@
   <inertial>
     <origin xyz="0.017451641868345052 0.011000000017253497 0.030092246470602525" rpy="0 0 0"/>
-    <mass value="0.5685307980275295"/>
-    <inertia ixx="0.000196" iyy="0.000234" izz="0.000133" ixy="0.0" iyz="0.0" ixz="-7e-06"/>
+    <!-- mass from MX-64R spec sheet (robotis.com, 902-0065-000): 126g -->
+    <mass value="0.126"/>
+    <inertia ixx="4.344e-05" iyy="5.186e-05" izz="2.948e-05" ixy="0.0" iyz="0.0" ixz="-1.551e-06"/>
   </inertial>
   <visual>
@@ -47,6 +48,7 @@
   <inertial>
     <origin xyz="-0.017451641868345052 0.010999999982746273 0.030092246470602525" rpy="0 0 0"/>
-    <mass value="0.5685307980275295"/>
-    <inertia ixx="0.000196" iyy="0.000234" izz="0.000133" ixy="0.0" iyz="-0.0" ixz="7e-06"/>
+    <!-- mass from MX-64R spec sheet (robotis.com, 902-0065-000): 126g -->
+    <mass value="0.126"/>
+    <inertia ixx="4.344e-05" iyy="5.186e-05" izz="2.948e-05" ixy="0.0" iyz="-0.0" ixz="1.551e-06"/>
   </inertial>
   <visual>
@@ -107,6 +109,7 @@
   <inertial>
     <origin xyz="0.017300000017253583 -0.019207753529397596 0.017451641868345094" rpy="0 0 0"/>
-    <mass value="0.5685307980275295"/>
-    <inertia ixx="0.000234" iyy="0.000133" izz="0.000196" ixy="0.0" iyz="-7e-06" ixz="0.0"/>
+    <!-- mass from MX-64R spec sheet (robotis.com, 902-0065-000): 126g -->
+    <mass value="0.126"/>
+    <inertia ixx="5.186e-05" iyy="2.948e-05" izz="4.344e-05" ixy="0.0" iyz="-1.551e-06" ixz="0.0"/>
   </inertial>
   <visual>
@@ -147,6 +150,7 @@
   <inertial>
     <origin xyz="0.02362282770461404 1.947747047686965e-05 0.05189568925169269" rpy="0 0 0"/>
-    <mass value="0.24310181617070015"/>
-    <inertia ixx="0.00024" iyy="0.000289" izz="9.7e-05" ixy="0.0" iyz="0.0" ixz="1e-06"/>
+    <!-- mass measured: arm_v9_1 = 27g -->
+    <mass value="0.027"/>
+    <inertia ixx="2.666e-05" iyy="3.21e-05" izz="1.077e-05" ixy="0.0" iyz="0.0" ixz="1.11e-07"/>
   </inertial>
   <visual>
@@ -187,6 +191,7 @@
   <inertial>
     <origin xyz="0.015031845145486198 0.017984471617669542 0.014999999976589629" rpy="0 0 0"/>
-    <mass value="0.3395854409997755"/>
-    <inertia ixx="8.1e-05" iyy="5.9e-05" izz="9.6e-05" ixy="1e-06" iyz="-0.0" ixz="0.0"/>
+    <!-- mass from MX-28T spec sheet (robotis.com, 902-0067-000): 72g -->
+    <mass value="0.072"/>
+    <inertia ixx="1.717e-05" iyy="1.251e-05" izz="2.035e-05" ixy="2.12e-07" iyz="-0.0" ixz="0.0"/>
   </inertial>
   <visual>
@@ -227,6 +232,7 @@
   <inertial>
     <origin xyz="-0.007777999999573574 0.03999999999999991 -0.007778000000000118" rpy="0 0 0"/>
-    <mass value="0.1756574712319971"/>
-    <inertia ixx="0.000149" iyy="3.9e-05" izz="0.000149" ixy="-0.0" iyz="-0.0" ixz="-0.0"/>
+    <!-- mass measured: arm2_v2_1 = 21.7g -->
+    <mass value="0.0217"/>
+    <inertia ixx="1.841e-05" iyy="4.818e-06" izz="1.841e-05" ixy="-0.0" iyz="-0.0" ixz="-0.0"/>
   </inertial>
   <visual>
@@ -267,6 +273,7 @@
   <inertial>
     <origin xyz="0.015031845145486136 0.024284471617669556 0.008499999976589567" rpy="0 0 0"/>
-    <mass value="0.3395854409997755"/>
-    <inertia ixx="8.1e-05" iyy="5.9e-05" izz="9.6e-05" ixy="1e-06" iyz="-0.0" ixz="0.0"/>
+    <!-- mass from MX-28T spec sheet (robotis.com, 902-0067-000): 72g -->
+    <mass value="0.072"/>
+    <inertia ixx="1.717e-05" iyy="1.251e-05" izz="2.035e-05" ixy="2.12e-07" iyz="-0.0" ixz="0.0"/>
   </inertial>
   <visual>
@@ -307,6 +314,9 @@
   <inertial>
     <origin xyz="0.007777999999983611 0.01501142035517336 -0.0015451576233940778" rpy="0 0 0"/>
-    <mass value="0.3222277062125533"/>
-    <inertia ixx="0.000105" iyy="0.000164" izz="0.000128" ixy="0.0" iyz="0.0" ixz="0.0"/>
+    <!-- TODO: measured mass is from racket_joint_v9_1 (13.3g + 13.2g = 26.5g); this link's mesh is
+         still racket_joint_v8_1 and the STL shape looked different from the v9 parts weighed.
+         Re-verify mass/inertia once the v9 mesh replaces v8 in this URDF. -->
+    <mass value="0.0265"/>
+    <inertia ixx="8.635e-06" iyy="1.349e-05" izz="1.053e-05" ixy="0.0" iyz="0.0" ixz="0.0"/>
   </inertial>
   <visual>
@@ -327,6 +337,7 @@
   <inertial>
     <origin xyz="6.7342507438505894e-15 -0.006399999999999961 -0.046816094811444026" rpy="0 0 0"/>
-    <mass value="2.4030890000623666"/>
-    <inertia ixx="0.008861" iyy="0.011682" izz="0.002911" ixy="-0.0" iyz="0.0" ixz="-0.0"/>
+    <!-- mass measured: pingpong_paddle_v5_1 = 172.9g (with protective film still on, not peeled) -->
+    <mass value="0.1729"/>
+    <inertia ixx="0.0006375" iyy="0.0008405" izz="0.0002094" ixy="-0.0" iyz="0.0" ixz="-0.0"/>
   </inertial>
   <visual>
